Commit message: In simulation package added a rectangular plate (representing a table) under the robot model

File: src/ur5e_leitungssatz_sim/urdf/ur5e_gripper.urdf.xacro (robot description, xacro)
@@ -7,4 +7,6 @@
    <xacro:include filename="$(find ur5e_leitungssatz_sim)/urdf/camera.xacro"/>
    <xacro:include filename="$(find ur5e_leitungssatz_sim)/urdf/ur5e_macro.xacro"/>
+   <!--Import table model-->
+   <xacro:include filename="$(find ur5e_leitungssatz_sim)/urdf/table.urdf.xacro"/>
    <!-- possible 'ur_type' values: ur3, ur3e, ur5, ur5e, ur7e, ur10, ur10e, ur12e, ur16e, ur15, ur20, ur30 -->
    <!-- the default value should raise an error in case this was called without defining the type -->
@@ -83,5 +85,5 @@
      name="$(arg name)"
      tf_prefix="$(arg tf_prefix)"
-     parent="world"
+     parent="table_link"
      joint_limits_parameters_file="$(arg joint_limit_params)"
      kinematics_parameters_file="$(arg kinematics_params)"
@@ -117,5 +119,5 @@
      trajectory_port="$(arg trajectory_port)"
      >
-     <origin xyz="0 0 0.8" rpy="0 0 0" />          <!-- position robot in the world -->
+     <origin xyz="0 0 0" rpy="0 0 0" />       <!--position robot in the world -->
    </xacro:ur_robot>
    <xacro:if value="$(arg sim_gazebo)">
@@ -144,4 +146,10 @@
   <!-- Import macros -->
   <xacro:include filename="$(find ur5e_leitungssatz_sim)/urdf/robotiq_gripper_macro.urdf.xacro" />
+  <!-- Fix UR5e on table -->
+  <!-- <joint name="table_to_ur5_base" type="fixed">
+    <parent link="table_link"/>
+    <child link="base_link"/>
+    <origin xyz="0 0 0.05" rpy="0 0 0"/>
+  </joint> -->
   <!-- <link name="world" /> -->
   <xacro:robotiq_gripper name="RobotiqGripperHardwareInterface" prefix="" parent="tool0" use_fake_hardware="$(arg use_fake_hardware)" com_port="$(arg com_port)" sim_gazebo="$(arg sim_gazebo)">
